File: KiCad/KiCad.kicad_pcb (KiCad board)
At the start: 2 copper layers, 130 x 54 mm, 16 parts, among them J1 EXT1, J2 EXT1, J3 EXT1, J4 Conn_01x20, J5 Conn_01x20, SW1 RESET, U1 Pico, U2 Pico

Commit message: update new PCB
Parts:
- added J6: Conn_01x03_Pin, Connector_PinHeader_2.54mm:PinHeader_1x03_P2.54mm_Vertical, F.Cu at (73.0, 84.5)
- SW1: value RESET -> SW_Push
Routing:
- net Net-(J6-Pin_3): track 78.1 -> 138.6 mm
- net Net-(J6-Pin_1): track 81.0 -> 135.4 mm, vias 0 -> 1
- net GND: track 419.9 -> 461.3 mm
- net /RUN: track 127.0 -> 121.6 mm
Other:
- board text added: "PICO PROBE DEBUG BOARD JP3SRS REL 2023/05/26 https://github.com/ngc6589"
- board text removed: "PICO PROBE DEBUG BOARD JP3SRS REL 2022/10/02 https://github.com/ngc6589"

Commit message: update board revision
Parts:
- added J7: 9-pin Cortex-M, Connector_PinHeader_1.27mm:PinHeader_2x05_P1.27mm_Vertical_SMD, F.Cu at (75.1, 86.9)
- SW1: value SW_Push -> RESET
- moved J6 5.05 mm to (73.0, 79.5)
- moved JP4 4.54 mm to (78.0, 74.8)
- moved JP3 4.54 mm to (73.0, 74.8)
- moved JP1 2.85 mm to (78.0, 65.2)
- moved JP2 2.85 mm to (73.0, 65.2)
- moved SW1 1.52 mm to (71.7, 93.5)
Routing:
- net /3V3: track 116.6 -> 199.4 mm
- net GND: track 461.3 -> 477.5 mm
- net Net-(J6-Pin_3): track 138.6 -> 148.2 mm, vias 0 -> 2
- net /RUN: track 121.6 -> 129.2 mm
- net Net-(JP2-B): track 14.6 -> 18.1 mm
- net Net-(JP3-B): track 22.1 -> 18.7 mm
- net /GP0: track 133.3 -> 136.5 mm
- net Net-(JP1-B): track 7.10 -> 9.96 mm
- net Net-(JP4-B): track 15.2 -> 12.6 mm
- net /GP1: track 123.8 -> 126.2 mm
- net Net-(J6-Pin_1): track 135.4 -> 136.0 mm, vias 1 -> 2
Other:
- board text added: "PICO PROBE DEBUG BOARD JP3SRS REL 2023/08/29 https://github.com/ngc6589"
- board text removed: "PICO PROBE DEBUG BOARD JP3SRS REL 2023/05/26 https://github.com/ngc6589"
