File: KiCad/KiCad.kicad_sch (KiCad schematic)
At the start: 16 parts, among them J1 EXT1, J2 EXT1, J3 EXT1, J4 Conn_01x20, J5 Conn_01x20, SW1 SW_Push, U1 Pico, U2 Pico

Commit message: update new PCB
Parts:
- added J6: Conn_01x03_Pin, Connector_PinHeader_2.54mm:PinHeader_1x03_P2.54mm_Vertical, symbol Connector:Conn_01x03_Pin
Connections:
- net GND: now also J6.2 (Pin_2)
- net at JP4.1 (A), U1.43 (SWDIO): now also J6.3 (Pin_3)
- net at JP3.1 (A), U1.41 (SWCLK): now also J6.1 (Pin_1)

Commit message: update board revision
Parts:
- added J7: 9-pin Cortex-M, Connector_PinHeader_1.27mm:PinHeader_2x05_P1.27mm_Vertical_SMD, symbol Connector_Generic:Conn_02x05_Odd_Even
- SW1: value SW_Push -> RESET
Connections:
- net 3V3: now also J7.1 (Pin_1)
- net GND: now also J7.3 (Pin_3), J7.5 (Pin_5)
- net RUN: now also J7.10 (Pin_10)
- net at J6.3 (Pin_3), JP4.1 (A), U1.43 (SWDIO): now also J7.2 (Pin_2)
- net at J6.1 (Pin_1), JP3.1 (A), U1.41 (SWCLK): now also J7.4 (Pin_4)
- no-connect marks 30 -> 34
Other:
- company: (none) -> Masahiro Kusunoki JP3SRS
- title: (none) -> Raspberry Pi Pico IO Expansion
